Commit message: position_control

File: src/gluon/urdf/gluon.urdf (robot description, URDF)
Before this commit: robot gluon, 8 links, 7 joints
Links:
- removed link dummy
- added link world
Joints:
- removed joint dummy_joint
- added joint world_fix: type fixed, parent world, child base_link, origin xyz=0 0 0.1 rpy=0 0 0
